File: hardware/_saved_prototype.sch (KiCad schematic (older format))
At the start: 95 parts, among them J1 CONN_02X20, SW1 SW_Push, SW10 SW_Push, SW11 SW_Push, SW12 SW_Push, SW13 SW_Push, SW14 SW_Push, SW15 SW_Push, SW16 SW_Push, SW17 SW_Push, SW18 SW_Push, SW19 SW_Push, SW2 SW_Push, SW20 SW_Push, SW21 SW_Push, SW22 SW_Push, SW23 SW_Push, SW24 SW_Push, SW25 SW_Push, SW26 SW_Push, SW3 SW_Push, SW4 SW_Push, SW5 SW_Push, SW6 SW_Push, SW7 SW_Push, SW8 SW_Push, SW9 SW_Push, U1 TLC5916, U10 SN74HC165N, U11 TLC5916, U2 TLC5916, U3 TLC5916, U4 SN74HC165N, U5 SN74HC165N, U6 TLC5916, U7 TLC5916, U8 TLC5916, U9 SN74HC165N

Commit message: Added more pcb stuff
Parts:
- D1, D10, D11, D12, D13, D14, D15, D16, D2, D3, D4, D5, D6, D7, D8, D9: footprint (none) -> piquantum-footprints:LED_D5.0mm-4
- D17, D18, D19, D20, D21, D22, D23, D24: footprint (none) -> piquantum-footprints:LED_D5.0mm
- J1: footprint (none) -> piquantum-footprints:IDC_Header_Straight_40pins
- R1, R2, R5, R6: footprint (none) -> piquantum-footprints:R_Axial_DIN0204_L3.6mm_D1.6mm_P7.62mm_Horizontal
- R10, R11, R12, R13, R14, R15, R16, R17, R18, R19, R20, R21, R22, R23, R24, R25, R26, R3, R4, R7, R8, R9: value R -> 2k7; footprint (none) -> piquantum-footprints:R_Axial_DIN0204_L3.6mm_D1.6mm_P7.62mm_Horizontal
- RV1, RV2, RV3, RV4, RV5, RV6, RV7: footprint (none) -> piquantum-footprints:Vishay_Trimmer_Through_Hole_2.54mm
- SW1, SW10, SW11, SW12, SW13, SW14, SW15, SW16, SW17, SW18, SW19, SW2, SW20, SW21, SW22, SW23, SW24, SW25, SW26, SW3, SW4, SW5, SW6, SW7, SW8, SW9: footprint (none) -> piquantum-footprints:SW_PUSH_5mm_h7.5mm
- U1, U10, U11, U2, U3, U4, U5, U6, U7, U8, U9: footprint (none) -> piquantum-footprints:DIP-16_W7.62mm_LongPads
