File: hardware/noname-03-05-2019.kicad_pcb (KiCad board)
At the start: 2 copper layers, 200 x 200 mm, 111 parts, among them J1 CONN_02X20, SW1 SW_Push, SW10 SW_Push, SW11 SW_Push, SW12 SW_Push, SW13 SW_Push, SW14 SW_Push, SW15 SW_Push, SW16 SW_Push, SW17 SW_Push, SW18 SW_Push, SW19 SW_Push, SW2 SW_Push, SW20 SW_Push, SW21 SW_Push, SW22 SW_Push, SW23 SW_Push, SW24 SW_Push, SW25 SW_Push, SW26 SW_Push, SW3 SW_Push, SW4 SW_Push, SW5 SW_Push, SW6 SW_Push, SW7 SW_Push, SW8 SW_Push, SW9 SW_Push, U1 TLC5916, U10 SN74HC165N, U11 TLC5916, U2 TLC5916, U3 TLC5916, U4 SN74HC165N, U5 SN74HC165N, U6 TLC5916, U7 TLC5916, U8 TLC5916, U9 SN74HC165N

Commit message: Added more pcb stuff
Parts:
- removed Q** (x16): qubit_label, piquantum-footprints:qubit_label
- moved R18 264.7 mm to (341.6, 85.1)
- moved R4 261.4 mm to (341.6, 57.1)
- moved RV1 255.2 mm to (327.7, 156.2)
- moved R3 250.7 mm to (346.7, 64.8)
- moved R20 243.7 mm to (322.6, 55.9)
- moved R17 243.2 mm to (313.7, 104.1)
- moved R19 240.8 mm to (303.5, 54.6)
- moved R26 237.5 mm to (341.6, 109.2)
- moved R21 222.0 mm to (299.7, 87.6)
- moved R1 200.9 mm to (325.1, 71.1), turned to 0 degrees
- moved R24 199.1 mm to (312.4, 64.8)
- moved R2 199.0 mm to (304.8, 72.4)
- moved SW25 194.0 mm to (92.7, 87.6)
- moved R5 189.2 mm to (330.2, 86.4)
- moved R22 187.5 mm to (334.0, 123.2)
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