File: hardware/prototype.kicad_pcb (KiCad board)
At the start: 2 copper layers, 200 x 200 mm, 111 parts, among them J1 CONN_02X20, SW1 SW_Push, SW10 SW_Push, SW11 SW_Push, SW12 SW_Push, SW13 SW_Push, SW14 SW_Push, SW15 SW_Push, SW16 SW_Push, SW17 SW_Push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

Commit message: More pcb stuff
Parts:
- renumbered Q** to Q1
