File: hardware/prototype.kicad_pcb (KiCad board)
At the start: 2 copper layers, 200 x 200 mm, 95 parts, among them J1 CONN_02X20, SW1 SW_Push, SW10 SW_Push, SW11 SW_Push, SW12 SW_Push, SW13 SW_Push, SW14 SW_Push, SW15 SW_Push, SW16 SW_Push, SW17 SW_Push, SW18 SW_Push, SW19 SW_Push, SW2 SW_Push, SW20 SW_Push, SW21 SW_Push, SW22 SW_Push, SW23 SW_Push, SW24 SW_Push, SW25 SW_Push, SW26 SW_Push, SW3 SW_Push, SW4 SW_Push, SW5 SW_Push, SW6 SW_Push, SW7 SW_Push, SW8 SW_Push, SW9 SW_Push, U1 TLC5916, U10 SN74HC165N, U11 TLC5916, U2 TLC5916, U3 TLC5916, U4 SN74HC165N, U5 SN74HC165N, U6 TLC5916, U7 TLC5916, U8 TLC5916, U9 SN74HC165N

Commit message: PCB stuff
Parts:
- moved R22 19.9 mm to (181.4, 218.0)
- moved R23 19.9 mm to (195.4, 218.0)
- moved R24 19.9 mm to (209.4, 218.0)
- moved R25 19.9 mm to (223.3, 218.0)
- moved U9 15.0 mm to (69.8, 192.0)
- moved SW17 15.0 mm to (84.1, 223.0)
- moved R17 15.0 mm to (84.1, 218.0)
- moved U10 14.8 mm to (157.0, 204.0)
- moved D17 12.9 mm to (184.0, 194.0)
- moved D21 12.7 mm to (184.0, 207.0)
- moved D20 11.9 mm to (226.0, 194.0)
- moved D24 11.7 mm to (226.0, 207.0)
- moved SW18 11.0 mm to (102.0, 223.0)
- moved R18 11.0 mm to (102.0, 218.0)
- moved D18 10.0 mm to (198.0, 194.0)
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Connections:
- U11 pad 1: Net-(RV7-Pad3) -> GND
- U11 pad 15: GND -> Net-(RV7-Pad3)
Routing:
- net Net-(D1-Pad3): track 1141.7 -> 0.00 mm
- net GND: track 1125.7 -> 0.00 mm
- net Net-(J1-Pad23): track 597.2 -> 0.00 mm
- net Net-(J1-Pad11): track 440.1 -> 0.00 mm
- net Net-(J1-Pad12): track 424.2 -> 0.00 mm
- net Net-(J1-Pad33): track 369.9 -> 0.00 mm
- net Net-(R25-Pad1): track 176.2 -> 0.00 mm
- net Net-(U11-Pad2): track 160.3 -> 0.00 mm
- net Net-(J1-Pad21): track 152.5 -> 0.00 mm
- net Net-(U4-Pad9): track 133.8 -> 0.00 mm
- net Net-(U10-Pad9): track 104.4 -> 0.00 mm
- net Net-(R2-Pad1): track 93.6 -> 0.00 mm
- net Net-(R14-Pad1): track 92.7 -> 0.00 mm
- net Net-(D7-Pad4): track 85.6 -> 0.00 mm
- net Net-(R17-Pad1): track 84.7 -> 0.00 mm
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
Commit message: Added gerbers
Parts:
- added REF**: via, piquantum-footprints:via, F.Cu at (196.0, 125.0)
- added REF**: via, piquantum-footprints:via, F.Cu at (137.0, 176.0)
- added REF**: via, piquantum-footprints:via, F.Cu at (201.0, 56.0)
- added REF**: via, piquantum-footprints:via, F.Cu at (121.0, 87.0)
- added REF**: via, piquantum-footprints:via, F.Cu at (127.0, 148.0)
- added REF**: via, piquantum-footprints:via, F.Cu at (227.0, 101.0)
- added REF**: via, piquantum-footprints:via, F.Cu at (103.0, 142.0)
- added REF**: via, piquantum-footprints:via, F.Cu at (80.0, 99.0)
- added REF**: via, piquantum-footprints:via, F.Cu at (76.0, 130.0)
Routing:
- net Net-(D1-Pad3): track 0.00 -> 1196.3 mm
- net GND: track 0.00 -> 1160.8 mm
- net Net-(J1-Pad23): track 0.00 -> 587.8 mm
- net Net-(J1-Pad11): track 0.00 -> 446.9 mm
- net Net-(J1-Pad12): track 0.00 -> 408.8 mm
- net Net-(J1-Pad33): track 0.00 -> 362.1 mm
- net Net-(U11-Pad2): track 0.00 -> 185.1 mm
- net Net-(R25-Pad1): track 0.00 -> 179.8 mm
- net Net-(J1-Pad21): track 0.00 -> 137.7 mm
- net Net-(U4-Pad9): track 0.00 -> 133.9 mm
- net Net-(R15-Pad1): track 0.00 -> 101.8 mm, vias 0 -> 1
- net Net-(D10-Pad2): track 0.00 -> 96.5 mm
- net Net-(U10-Pad9): track 0.00 -> 94.2 mm
- net Net-(R14-Pad1): track 0.00 -> 93.5 mm
- net Net-(R17-Pad1): track 0.00 -> 93.2 mm
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- added copper zone on B.Cu, net GND
- added copper zone on F.Cu, net GND
Other:
- net class Default: clearance 0.2 -> 0.155; trace_width 0.25 -> 0.3
- rule trace_clearance: 0.2 -> 0.155
- board text added: "1"
- board text added: "10"
- board text added: "11"
- board text added: "12"
- board text added: "13"
- board text added: "14"
- board text added: "15"
- board text added: "16"
- board text added: "2"
- board text added: "3"
- board text added: "4"
- board text added: "5"
- board text added: "6"
- board text added: "7"
- board text added: "8"
- board text added: "9"
- board text added: "Oliver Thomas and John Scott, QETLabs, University of Bristol"
- board text added: "PiQuantum"
