File: hardware/grid-done.kicad_pcb (KiCad board)
At the start: 2 copper layers, 200 x 200 mm, 95 parts, among them J1 CONN_02X20, SW1 SW_Push, SW10 SW_Push, SW11 SW_Push, SW12 SW_Push, SW13 SW_Push, SW14 SW_Push, SW15 SW_Push, SW16 SW_Push, SW17 SW_Push, SW18 SW_Push, SW19 SW_Push, SW2 SW_Push, SW20 SW_Push, SW21 SW_Push, SW22 SW_Push, SW23 SW_Push, SW24 SW_Push, SW25 SW_Push, SW26 SW_Push, SW3 SW_Push, SW4 SW_Push, SW5 SW_Push, SW6 SW_Push, SW7 SW_Push, SW8 SW_Push, SW9 SW_Push, U1 TLC5916, U10 SN74HC165N, U11 TLC5916, U2 TLC5916, U3 TLC5916, U4 SN74HC165N, U5 SN74HC165N, U6 TLC5916, U7 TLC5916, U8 TLC5916, U9 SN74HC165N

Commit message: PCB stuff
Parts:
- moved U4 139.5 mm to (293.4, 109.2), turned to 180 degrees
- moved R10 30.0 mm to (183.0, 140.0)
- moved R11 30.0 mm to (183.0, 110.0)
- moved U5 6.55 mm to (154.9, 184.2), turned to 0 degrees
- moved RV1 1.38 mm to (88.9, 66.0)
- moved U2 0.94 mm to (87.6, 114.3)
- moved RV2 0.93 mm to (88.9, 109.2)
- moved U1 0.64 mm to (87.6, 71.1)
- moved U3 0.63 mm to (87.6, 157.5)
Routing:
- net Net-(D1-Pad3): track 1141.7 -> 0.00 mm
- net GND: track 1125.7 -> 0.00 mm
- net Net-(J1-Pad23): track 597.2 -> 0.00 mm
- net Net-(J1-Pad11): track 440.1 -> 0.00 mm
- net Net-(J1-Pad12): track 424.2 -> 0.00 mm
- net Net-(J1-Pad33): track 369.9 -> 0.00 mm
- net Net-(R25-Pad1): track 176.2 -> 0.00 mm
- net Net-(U11-Pad2): track 160.3 -> 0.00 mm
- net Net-(J1-Pad21): track 152.5 -> 0.00 mm
- net Net-(U4-Pad9): track 133.8 -> 0.00 mm
- net Net-(U10-Pad9): track 104.4 -> 0.00 mm
- net Net-(R2-Pad1): track 93.6 -> 0.00 mm
- net Net-(R14-Pad1): track 92.7 -> 0.00 mm
- net Net-(D7-Pad4): track 85.6 -> 0.00 mm
- net Net-(R17-Pad1): track 84.7 -> 0.00 mm
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