File: hardware/prototype.sch (KiCad schematic (older format))
At the start: 85 parts, among them J1 CONN_02X20, SW1 SW_Push, SW10 SW_Push, SW11 SW_Push, SW12 SW_Push, SW13 SW_Push, SW14 SW_Push, SW15 SW_Push, SW16 SW_Push, SW17 SW_Push, SW18 SW_Push, SW19 SW_Push, SW2 SW_Push, SW20 SW_Push, SW21 SW_Push, SW22 SW_Push, SW23 SW_Push, SW24 SW_Push, SW25 SW_Push, SW26 SW_Push, SW3 SW_Push, SW4 SW_Push, SW5 SW_Push, SW6 SW_Push, SW7 SW_Push, SW8 SW_Push, SW9 SW_Push, U1 TLC5916, U10 SN74HC165N, U2 TLC5916, U3 TLC5916, U4 SN74HC165N, U5 SN74HC165N, U6 TLC5916, U7 TLC5916, U8 TLC5916, U9 SN74HC165N

Commit message: Added more pcb stuff
Parts:
- added D17, D18, D19, D20, D21, D22, D23, D24: LED, symbol LED
- added RV7: POT, optojig-footprints:Vishay_Trimmer_Through_Hole_2.54mm, symbol POT
- added U11: TLC5916, symbol TLC5916
- D1, D10, D11, D12, D13, D14, D15, D16, D2, D3, D4, D5, D6, D7, D8, D9: symbol LED_RABG -> LED_RABG-RESCUE-prototype
- R1, R2, R5, R6: value R -> 2k7
- RV1, RV2, RV3, RV4, RV5, RV6: footprint (none) -> optojig-footprints:Vishay_Trimmer_Through_Hole_2.54mm
Connections:
- net GND: now also J1.6 (P6), U4.10 (SER), RV7.1, RV7.2, U11.15 (REXT)
- net at J1.1 (P1), SW1.1, SW10.1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: now also D1.3 (A), D10.3 (A), D11.3 (A), D12.3 (A), D13.3 (A), D14.3 (A), D15.3 (A), D16.3 (A), D2.3 (A), D3.3 (A), D4.3 (A), D5.3 (A), D6.3 (A), D7.3 (A), D8.3 (A), D9.3 (A), D17.2 (A), D18.2 (A), D19.2 (A), D20.2 (A), D21.2 (A), D22.2 (A), D23.2 (A), D24.2 (A), U11.16 (VDD); no longer D1.2 (A), D10.2 (A), D11.2 (A), D12.2 (A), D13.2 (A), D14.2 (A), D15.2 (A), D16.2 (A), D2.2 (A), D3.2 (A), D4.2 (A), D5.2 (A), D6.2 (A), D7.2 (A), D8.2 (A), D9.2 (A)
- net at J1.11 (P11), U1.4 (LE), U2.4 (LE)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: now also U11.4 (LE)
- net at J1.12 (P12), U1.13 (OE), U2.13 (OE)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: now also U11.13 (OE)
- net at J1.23 (P23), U1.3 (CLK), U10.2 (CLK)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: now also U11.3 (CLK)
- net at U1.10 (Out5): now also D5.2 (BK); no longer D5.3 (BK)
- net at U1.11 (Out6): now also D6.4 (RK); no longer D6.1 (RK)
- net at U1.12 (Out7): now also D6.1 (GK); no longer D6.4 (GK)
- net at U1.5 (Out0): now also D1.4 (RK); no longer D1.1 (RK)
- net at U1.6 (Out1): now also D1.1 (GK); no longer D1.4 (GK)
- net at U1.7 (Out2): now also D1.2 (BK); no longer D1.3 (BK)
- net at U1.8 (Out3): now also D5.4 (RK); no longer D5.1 (RK)
- net at U1.9 (Out4): now also D5.1 (GK); no longer D5.4 (GK)
- net at U2.10 (Out5): now also D3.2 (BK); no longer D3.3 (BK)
- net at U2.11 (Out6): now also D3.1 (GK); no longer D3.4 (GK)
- net at U2.12 (Out7): now also D3.4 (RK); no longer D3.1 (RK)
- net at U2.5 (Out0): now also D2.4 (RK); no longer D2.1 (RK)
- net at U2.6 (Out1): now also D2.1 (GK); no longer D2.4 (GK)
- net at U2.7 (Out2): now also D2.2 (BK); no longer D2.3 (BK)
- net at U2.8 (Out3): now also D6.2 (BK); no longer D6.3 (BK)
- net at U2.9 (Out4): now also D7.2 (BK); no longer D7.3 (BK)
- net at U3.10 (Out5): now also D4.2 (BK); no longer D4.3 (BK)
- net at U3.11 (Out6): now also D4.1 (GK); no longer D4.4 (GK)
- net at U3.12 (Out7): now also D4.4 (RK); no longer D4.1 (RK)
- net at U3.14 (SDO): now also U11.2 (SDI); no longer U8.2 (SDI)
- net at U3.5 (Out0): now also D7.1 (GK); no longer D7.4 (GK)
- net at U3.6 (Out1): now also D7.4 (RK); no longer D7.1 (RK)
- net at U3.7 (Out2): now also D8.2 (BK); no longer D8.3 (BK)
- net at U3.8 (Out3): now also D8.1 (GK); no longer D8.4 (GK)
- net at U3.9 (Out4): now also D8.4 (RK); no longer D8.1 (RK)
- net at U6.10 (Out5): now also D9.2 (BK); no longer D9.3 (BK)
- net at U6.11 (Out6): now also D10.4 (RK); no longer D10.1 (RK)
- net at U6.12 (Out7): now also D10.1 (GK); no longer D10.4 (GK)
- net at U6.5 (Out0): now also D13.4 (RK); no longer D13.1 (RK)
- net at U6.6 (Out1): now also D13.1 (GK); no longer D13.4 (GK)
- net at U6.7 (Out2): now also D13.2 (BK); no longer D13.3 (BK)
- net at U6.8 (Out3): now also D9.4 (RK); no longer D9.1 (RK)
- net at U6.9 (Out4): now also D9.1 (GK); no longer D9.4 (GK)
- net at U8.10 (Out5): now also D16.2 (BK); no longer D16.3 (BK)
- net at U8.11 (Out6): now also D16.1 (GK); no longer D16.4 (GK)
- net at U8.12 (Out7): now also D16.4 (RK); no longer D16.1 (RK)
- net at U8.5 (Out0): now also D11.1 (GK); no longer D11.4 (GK)
- net at U8.6 (Out1): now also D11.4 (RK); no longer D11.1 (RK)
- net at U8.7 (Out2): now also D12.2 (BK); no longer D12.3 (BK)
- net at U8.8 (Out3): now also D12.1 (GK); no longer D12.4 (GK)
- net at U8.9 (Out4): now also D12.4 (RK); no longer D12.1 (RK)
- net at U7.10 (Out5): now also D15.2 (BK); no longer D15.3 (BK)
- net at U7.11 (Out6): now also D15.1 (GK); no longer D15.4 (GK)
- net at U7.12 (Out7): now also D15.4 (RK); no longer D15.1 (RK)
- net at U7.5 (Out0): now also D14.4 (RK); no longer D14.1 (RK)
- net at U7.6 (Out1): now also D14.1 (GK); no longer D14.4 (GK)
- net at U7.7 (Out2): now also D14.2 (BK); no longer D14.3 (BK)
- net at U7.8 (Out3): now also D10.2 (BK); no longer D10.3 (BK)
- net at U7.9 (Out4): now also D11.2 (BK); no longer D11.3 (BK)
- new net: U11.14 (SDO), U8.2 (SDI)
- new net: RV7.3, U11.1 (GND)
- new net: D22.1 (K), U11.10 (Out5)
- new net: D23.1 (K), U11.11 (Out6)
- new net: D24.1 (K), U11.12 (Out7)
- new net: D17.1 (K), U11.5 (Out0)
- new net: D18.1 (K), U11.6 (Out1)
- new net: D19.1 (K), U11.7 (Out2)
- new net: D20.1 (K), U11.8 (Out3)
- new net: D21.1 (K), U11.9 (Out4)

Commit message: PCB stuff
Parts:
- D1, D10, D11, D12, D13, D14, D15, D16, D2, D3, D4, D5, D6, D7, D8, D9: footprint (none) -> piquantum-footprints:LED_D5.0mm-4
- D17, D18, D19, D20, D21, D22, D23, D24: footprint (none) -> piquantum-footprints:LED_D5.0mm
- J1: footprint (none) -> piquantum-footprints:IDC_Header_Straight_40pins
- R1, R2, R5, R6: footprint (none) -> piquantum-footprints:R_Axial_DIN0204_L3.6mm_D1.6mm_P7.62mm_Horizontal
- R10, R11, R12, R13, R14, R15, R16, R17, R18, R19, R20, R21, R22, R23, R24, R25, R26, R3, R4, R7, R8, R9: value R -> 2k7; footprint (none) -> piquantum-footprints:R_Axial_DIN0204_L3.6mm_D1.6mm_P7.62mm_Horizontal
- RV1, RV2, RV3, RV4, RV5, RV6, RV7: footprint optojig-footprints:Vishay_Trimmer_Through_Hole_2.54mm -> piquantum-footprints:Vishay_Trimmer_Through_Hole_2.54mm
- SW1, SW10, SW11, SW12, SW13, SW14, SW15, SW16, SW17, SW18, SW19, SW2, SW20, SW21, SW22, SW23, SW24, SW25, SW26, SW3, SW4, SW5, SW6, SW7, SW8, SW9: footprint (none) -> piquantum-footprints:SW_PUSH_5mm_h7.5mm
- U1, U10, U11, U2, U3, U4, U5, U6, U7, U8, U9: footprint (none) -> piquantum-footprints:DIP-16_W7.62mm_LongPads

Commit message: PCB stuff
Connections:
- net GND: now also U11.1 (GND); no longer U11.15 (REXT)
- net at RV7.3: now also U11.15 (REXT); no longer U11.1 (GND)
Other:
- moved on the sheet: RV7
Changed lines of the file:
@@
 L GND #PWR026
 U 1 1 5CCC49F7
-P 9900 10950
-F 0 "#PWR026" H 9900 10700 50  0001 C CNN
-F 1 "GND" H 9900 10800 50  0000 C CNN
-F 2 "" H 9900 10950 50  0001 C CNN
-F 3 "" H 9900 10950 50  0001 C CNN
-	1    9900 10950
-	-1   0    0    -1
+P 9700 10950
+F 0 "#PWR026" H 9700 10700 50  0001 C CNN
+F 1 "GND" H 9700 10800 50  0000 C CNN
+F 2 "" H 9700 10950 50  0001 C CNN
+F 3 "" H 9700 10950 50  0001 C CNN
+	1    9700 10950
+	1    0    0    -1
 $EndComp
 $Comp
 L POT RV7
 U 1 1 5CCC49FD
-P 9700 10550
-F 0 "RV7" V 9525 10550 50  0000 C CNN
-F 1 "POT" V 9600 10550 50  0000 C CNN
-F 2 "piquantum-footprints:Vishay_Trimmer_Through_Hole_2.54mm" H 9700 10550 50  0001 C CNN
-F 3 "" H 9700 10550 50  0001 C CNN
-	1    9700 10550
-	1    0    0    1
+P 9900 10550
+F 0 "RV7" V 9725 10550 50  0000 C CNN
+F 1 "POT" V 9800 10550 50  0000 C CNN
+F 2 "piquantum-footprints:Vishay_Trimmer_Through_Hole_2.54mm" H 9900 10550 50  0001 C CNN
+F 3 "" H 9900 10550 50  0001 C CNN
+	1    9900 10550
+	-1   0    0    1
 $EndComp
 $Comp
@@
 Connection ~ 7900 10800
 Connection ~ 8200 10800
-Connection ~ 9900 10550
-Wire Wire Line
-	9850 10550 9900 10550
-Connection ~ 9900 10750
-Wire Wire Line
-	9900 10750 9700 10750
-Wire Wire Line
-	9700 10750 9700 10700
-Wire Wire Line
-	9550 10550 9500 10550
-Wire Wire Line
-	9900 10300 9900 10950
-Wire Wire Line
-	9700 10300 9700 10400
+Connection ~ 9700 10550
+Wire Wire Line
+	9750 10550 9700 10550
+Connection ~ 9700 10750
+Wire Wire Line
+	9700 10750 9900 10750
+Wire Wire Line
+	9900 10750 9900 10700
+Wire Wire Line
+	10050 10550 10100 10550
+Wire Wire Line
+	9700 10300 9700 10950
+Wire Wire Line
+	9900 10300 9900 10400
 Connection ~ 8500 8850
 Wire Wire Line
